File: Pneumatics Control Unit V1.1/Pneumatics Control Unit V1.kicad_sch (KiCad schematic)
At the start: 44 parts

Commit message: Switching linear 3.3 to switching 3.3
Parts:
- removed U?: NCP1117LPST33T3G, SOT223-3_ONS, symbol 3.3:NCP1117LPST33T3G
- added C?: 6.8n, Capacitor_SMD:C_0805_2012Metric_Pad1.18x1.45mm_HandSolder, symbol Device:C
- added C?: 0.01u, Capacitor_SMD:C_0805_2012Metric_Pad1.18x1.45mm_HandSolder, symbol Device:C
- added C? (x2): 100u, Capacitor_SMD:C_0805_2012Metric_Pad1.18x1.45mm_HandSolder, symbol Device:C
- added CR?: MBRS130L, DIODE_DO214AA, symbol MBRS130L:MBRS130L
- added L?: 50u, symbol pspice:INDUCTOR
- added R? (x3): 10000, Resistor_SMD:R_0805_2012Metric_Pad1.20x1.40mm_HandSolder, symbol Device:R_US
- added U?: MIC2178-3.3YWM, SOICW-20LD-PL-1_MCH, symbol 3.3Sw:MIC2178-3.3YWM
Connections:
- net 3.3V: now also C?.1, L?.2, U?.12 (FB); no longer J?.11 (~{BOOT}), J?.2 (3.3V), J?.4 (3.3V_EN), J?.6 (~{RESET}), J?.72 (RTC_3V), J?.74 (3.3V)
- net 5V: no longer J?.2 (Pin_2), J?.2 (Pin_2), J?.2 (Pin_2), J?.2 (Pin_2), J?.2 (Pin_2), J?.2 (Pin_2), J?.2 (Pin_2), J?.2 (Pin_2), U?.1 (VCC)
- net GND: now also C?.1, C?.2, C?.2, C?.2, R?.2, U?.10 (*PWM), U?.14 (SGND), U?.15 (SGND), U?.16 (SGND), U?.17 (SGND), U?.18 (SYNC), U?.4 (PGND), U?.5 (PGND), U?.6 (PGND)
- net RS485_B_12V: now also C?.2, R?.2, U?.1 (VIN), U?.2 (VIN), U?.20 (EN), U?.9 (VIN)
- new net: C?.1, R?.1, U?.19 (BIAS)
- new net: CR?.1, L?.1, U?.3 (SW), U?.8 (SW)
- new net: C?.1, R?.2
- new net: R?.1, U?.13 (COMP)
- new net: R?.1, U?.11 (PWRGD)
- new net +3V3: J?.11 (~{BOOT}), J?.2 (3.3V), J?.4 (3.3V_EN), J?.6 (~{RESET}), J?.72 (RTC_3V), J?.74 (3.3V), U?.1 (VCC)
- new net +5V: J?.2 (Pin_2), J?.2 (Pin_2), J?.2 (Pin_2), J?.2 (Pin_2), J?.2 (Pin_2), J?.2 (Pin_2), J?.2 (Pin_2), J?.2 (Pin_2)
Other:
- note added: "Power"
- moved on the sheet: D?, H1, H2, H3, J?, MOSFET?, U?, U?B

Commit message: Cleaning
Parts:
- removed U?: MDT420M02001, MDT420M02001_AMP, symbol m.2:MDT420M02001
Changed lines of the file:
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@@
     (pin "1")
-  )
-  (symbol (lib_id "m.2:MDT420M02001") (at 145.161 116.205 0) (mirror y) (unit 2)
-    (in_bom yes) (on_board yes) (fields_autoplaced)
-    (property "Reference" "U?" (id 0) (at 124.841 105.664 0)
-      (effects (font (size 1.524 1.524)))
-    )
-    (property "Value" "MDT420M02001" (id 1) (at 124.841 109.474 0)
-      (effects (font (size 1.524 1.524)))
-    )
-    (property "Footprint" "MDT420M02001_AMP" (id 2) (at 165.481 107.569 0)
-      (effects (font (size 1.524 1.524)) hide)
-    )
-    (property "Datasheet" "" (id 3) (at 145.161 116.205 0)
-      (effects (font (size 1.524 1.524)))
-    )
-    (pin "2")
-    (pin "20")
-    (pin "21")
-    (pin "22")
-    (pin "23")
-    (pin "24")
-    (pin "25")
-    (pin "26")
-    (pin "27")
-    (pin "28")
-    (pin "29")
-    (pin "3")
-    (pin "30")
-    (pin "31")
-    (pin "32")
-    (pin "33")
-    (pin "34")
-    (pin "35")
-    (pin "36")
-    (pin "37")
-    (pin "38")
-    (pin "39")
-    (pin "4")
-    (pin "40")
-    (pin "41")
-    (pin "42")
-    (pin "43")
-    (pin "44")
-    (pin "45")
-    (pin "46")
-    (pin "47")
-    (pin "48")
-    (pin "49")
-    (pin "5")
-    (pin "50")
-    (pin "51")
-    (pin "52")
-    (pin "53")
-    (pin "54")
-    (pin "55")
-    (pin "56")
-    (pin "57")
-    (pin "58")
-    (pin "6")
-    (pin "67")
-    (pin "68")
-    (pin "69")
-    (pin "7")
-    (pin "70")
-    (pin "71")
-    (pin "72")
-    (pin "73")
-    (pin "74")
-    (pin "75")
-    (pin "8")
-    (pin "9")
   )
   (symbol (lib_id "power:+5V") (at 363.093 209.296 0) (unit 1)
@@
       (reference "U?") (unit 1) (value "MC78M05CDTRKG") (footprint "DPAK-3_ONS")
     )
-    (path "/a0fc109e-39e3-4b9b-bb0a-dce49a5ef63b"
-      (reference "U?") (unit 2) (value "MDT420M02001") (footprint "MDT420M02001_AMP")
-    )
-  )
+  )
