File: Pneumatics Control Unit Pin (Senior Design)/Pneumatics Control Unit Pinned.kicad_sch (KiCad schematic)
At the start: 87 parts

Commit message: Senior Update
Parts:
- removed C1, C10, C11, C12, C13, C14, C15, C2, C3, C4, C5, C6, C7, C8, C9: (no value), symbol Device:C
- removed C18, C19, C20, C21, C22, C23, C24, C27, C29, C30: (no value), symbol Samsung Cap 22u:CL21A226MQQNNNF
- removed C?: CL21A226MQQNNNF, symbol Samsung Cap 22u:CL21A226MQQNNNF
- removed C?: 0.1u, Capacitor_SMD:C_0805_2012Metric_Pad1.18x1.45mm_HandSolder, symbol Device:C
- removed C?: 6.8n, Capacitor_SMD:C_0805_2012Metric_Pad1.18x1.45mm_HandSolder, symbol Device:C
- removed C?: 0.01u, Capacitor_SMD:C_0805_2012Metric_Pad1.18x1.45mm_HandSolder, symbol Device:C
- removed C?: 1u, Capacitor_SMD:C_0805_2012Metric_Pad1.18x1.45mm_HandSolder, symbol Device:C
- removed CR?: MBRS130L, symbol MBRS130L Diode:MBRS130L
- removed D10, D11, D12, D3, D4, D5, D6, D7, D8, D9: (no value), symbol Device:D_TVS_x2_AAC
- removed J10, J5, J6, J7, J8, J9: (no value), symbol Connector:Conn_01x02_Male
- removed L?: LB3218T330KV, symbol Taiyo Inductor 33uh:LB3218T330KV
- removed R1, R2, R3, R4: (no value), symbol Device:R_US
- removed R?: 20k, Resistor_SMD:R_0805_2012Metric_Pad1.20x1.40mm_HandSolder, symbol Device:R_US
- removed R? (x2): 10k, Resistor_SMD:R_0805_2012Metric_Pad1.20x1.40mm_HandSolder, symbol Device:R_US
- added C1, C10, C17, C2, C3, C8, C9: 1u, 1 uF Cap:C1608X7R1C105K080AC, symbol 1 uF Cap:C1608X7R1C105K080AC
- added C11, C12, C15, C28, C4, C5, C6, C7: 0.1u, 0.1 uF Cap:0402YC104KAT2A, symbol 0.1 uF Cap:0402YC104KAT2A
- added C13, C14: 10n, 10 nF Cap:0402YC103KAT2A, symbol 10 nF Cap:0402YC103KAT2A
- added C16, C18, C19, C20, C21, C22, C23, C24, C26, C29, C30: 22u, 22 uF Cap:CL21A226MQQNNNE, symbol 22 uF Cap:CL21A226MQQNNNE
- added C25: 0.01u, 0.01 uF cap:CL05B103KO5NNNC, symbol 0.01 uF Cap:CL05B103KO5NNNC
- added C27: 6.8n, 6.8 nF Cap:0402B682K500CT, symbol 6.8 nF Cap:0402B682K500CT
- added D10: CDBA340-HF, CDBA340-HF Diode:CDBA340-HF, symbol CDBA340-HF Diode:CDBA340-HF
- added D11, D12, D13, D3, D4, D5, D6, D7, D8, D9: PESD1FLEX,215, Dual Diode:PESD1FLEX215, symbol Dual Diode:PESD1FLEX,215
- added J10: I2C 2, symbol Connector:Conn_01x05_Male
- added J14, J15, J16, J17, J18, J19: Conn_01x02_Male, Connector_PinSocket_2.54mm:PinSocket_1x02_P2.54mm_Vertical, symbol Connector:Conn_01x02_Male
- added J20: Encoder 1 - CCW, symbol Connector:Conn_01x03_Female
- added J21, J23: (no value), symbol Connector:Conn_01x03_Female
- added J22: Encoder 1 - CW, symbol Connector:Conn_01x03_Female
- added J5: SPI 0, symbol Connector:Conn_01x12_Male
- added J6: SPI 1, symbol Connector:Conn_01x04_Male
- added J7: GPIO, symbol Connector:Conn_01x10_Male
- added J8: I2C 0, symbol Connector:Conn_01x05_Male
- added J9: I2C 1, symbol Connector:Conn_01x05_Male
- added L1: 33u, 33 uH Inductor:LB3218T330K, symbol 33 uH Inductor:LB3218T330K
- added R1, R2, R3, R4: 10, 10 Res:RNCP0603FTD10R0, symbol 10 Res:RNCP0603FTD10R0
- added R5: 20k, 20K Res:SR1-0805-320, symbol 20K Res:SR1-0805-320
- added R6, R7: 10K, 10K Res:SR1-0603-310, symbol 10K Res:SR1-0603-310
- D1: renamed from D?; value (none) -> PESD1FLEX,215
- H1, H2, H3, H4: value (none) -> MountingHole; footprint (none) -> MountingHole:MountingHole_2.5mm
- J1: value (none) -> RX_PORT; footprint (none) -> RS485:RS485
- J11, J12, J13, J4: value (none) -> Conn_01x02_Male; footprint (none) -> Connector_PinSocket_2.54mm:PinSocket_1x02_P2.54mm_Vertical
- J2: value (none) -> TX_PORT; footprint (none) -> RS485:RS485
- J3: value (none) -> 87583-2010BLF; footprint (none) -> USB 2.0 Type A:87583-2010BLF
- MOSFET1: renamed from MOSFET?; value (none) -> SSM3K7002KFU; footprint (none) -> Toshiba MOSFET:SSM3K7002KFU
- P1: value (none) -> J1B1211CCD; footprint (none) -> Ethernet:J1B1211CCD; Price None -> $3.78; Source (none) -> https://www.digikey.com/en/products/detail/wiznet/J1B1211CC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
- U1, U2, U3: value (none) -> MC78M05CDTRKG; footprint (none) -> 12V5V Regulator:MC78M05CDTRKG; Price (none) -> $0.54; Source (none) -> https://www.digikey.com/en/products/detail/onsemi/MC78M05CD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
- U4: value (none) -> Teensy4.1; footprint (none) -> Teensy:Teensy41; Price (none) -> $26.85; Source (none) -> https://www.pjrc.com/store/teensy41.html
- U5, U6: value (none) -> 74AXP2T3407GSX; footprint (none) -> Nexperia Level Shifter:74AXP2T3407GSX; Price (none) -> $0.64; Source (none) -> https://www.digikey.com/en/products/detail/nexperia-usa-inc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
- U7: renamed from U?; value (none) -> ISL83490IBZ; footprint (none) -> RS485 To UART:ISL83490IBZ
- U8: renamed from U?; value (none) -> MIC2178-3.3YWM; footprint (none) -> 33SW:MIC2178-33YWM; Price (none) -> $8.01; Source (none) -> https://www.digikey.com/en/products/detail/microchip-techno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
- gave numbers to parts that had none: 10
Connections:
- net 220uF is gone; now on net +3V3: U8.12 (FB)
- net V_IN is gone; now on net +5V: U4.48 (VIN)
- net Encoder_0_CCW: now also J20.2 (Pin_2)
- net Encoder_0_CW: now also J22.2 (Pin_2)
- net Encoder_1_CCW: now also J21.2 (Pin_2)
- net Encoder_1_CW: now also J23.2 (Pin_2)
- net GND: now also U7.4 (GND), C1.1, C10.1, C11.1, C12.1, C13.1, C14.1, C15.1, C16.1, C17.1, C18.1, C19.1, C2.1, C20.1, C21.1, C22.1, C23.1, C24.1, C25.2, C26.1, C27.1, C28.1, C29.1, C3.1, C30.1, C4.1, C5.1, C6.1, C7.1, C8.1, C9.1, D10.2, D11.3, D12.3, D13.3, D3.3, D4.3, D5.3, D6.3, D7.3, D8.3, D9.3, J10.1 (Pin_1), J20.3 (Pin_3), J21.3 (Pin_3), J22.3 (Pin_3), J23.3 (Pin_3), J8.1 (Pin_1), J9.1 (Pin_1), R7.2
- net GPIO_0: now also D3.1
- net GPIO_1: now also D7.1
- net GPIO_10: now also J7.1 (Pin_1)
- net GPIO_11: now also J7.2 (Pin_2)
- net GPIO_12: now also J7.3 (Pin_3)
- net GPIO_13: now also J7.4 (Pin_4)
- net GPIO_14: now also J7.5 (Pin_5)
- net GPIO_15: now also J7.6 (Pin_6)
- net GPIO_16: now also J7.7 (Pin_7)
- net GPIO_17: now also J7.8 (Pin_8)
- net GPIO_18: now also J7.9 (Pin_9)
- net GPIO_19: now also J7.10 (Pin_10)
- net GPIO_2: now also D11.1
- net GPIO_3: now also D4.1
- net GPIO_4: now also D8.1
- net GPIO_5: now also D12.1
- net GPIO_6: now also D5.1
- net GPIO_7: now also D9.1
- net GPIO_8: now also D13.1
- net GPIO_9: now also D6.1
- net I2C_0_SCL: now also J8.2 (Pin_2)
- net I2C_0_SDA: now also J8.3 (Pin_3)
- net I2C_1_SCL: now also J9.3 (Pin_3)
- net I2C_1_SDA: now also J9.2 (Pin_2)
- net I2C_2_SCL: now also J10.3 (Pin_3)
- net I2C_2_SDA: now also J10.2 (Pin_2)
- net RS485_A_12V: now also C16.2, C17.2, R5.2
- net RS485_B_12V: now also C1.2, C2.2, C3.2
- net SPI_0_CS_0: now also J5.9 (Pin_9)
- net SPI_0_CS_1: now also J5.5 (Pin_5)
- net SPI_0_CS_2: now also J5.1 (Pin_1)
- net SPI_0_MISO: now also J5.10 (Pin_10), J5.2 (Pin_2), J5.6 (Pin_6)
- net SPI_0_MOSI: now also J5.11 (Pin_11), J5.3 (Pin_3), J5.7 (Pin_7)
- net SPI_0_SCK: now also J5.12 (Pin_12), J5.4 (Pin_4), J5.8 (Pin_8)
- net SPI_1_CS: now also J6.1 (Pin_1)
- net SPI_1_MISO: now also J6.2 (Pin_2)
- net SPI_1_SCK: now also J6.4 (Pin_4)
- net at J13.1 (Pin_1): now also MOSFET4.3 (DRAIN), D6.2; no longer MOSFET10.3 (DRAIN)
- net +3V3: now reaches U4.15 (3V3)
- net +3V3: now also U4.46 (3V3), U5.1 (VCCI), U6.1 (VCCI), U7.1 (VCC), C18.2, C19.2, C20.2, C21.2, C22.2, C23.2, C24.2, C26.2, C28.2, C29.2, C30.2, J10.4 (Pin_4), J8.4 (Pin_4), J9.4 (Pin_4), L1.1
- net at J12.1 (Pin_1): now also MOSFET3.3 (DRAIN), D5.2; no longer MOSFET9.3 (DRAIN)
- net at U7.5 (Y): now also R4.2
- net at U7.6 (Z): now also R3.2
- net at U7.7 (B): now also R2.2
- net at U7.8 (A): now also R1.2
- net at D2.1, D2.2, J2.1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: now also C5.2, C7.2, R3.1, R4.1
- net at J4.1 (Pin_1), MOSFET1.3 (DRAIN): now also D3.2
- net +5V: now reaches U5.8 (VCCO), U6.8 (VCCO)
- net +5V: now also J11.2 (Pin_2), J12.2 (Pin_2), J13.2 (Pin_2), J3.4 (VCC), J4.2 (Pin_2), U1.3 (OUTPUT), U2.3 (OUTPUT), U3.3 (OUTPUT), C10.2, C11.2, C12.2, C13.2, C14.2, C8.2, C9.2, J10.5 (Pin_5), J14.2 (Pin_2), J15.2 (Pin_2), J16.2 (Pin_2), J17.2 (Pin_2), J18.2 (Pin_2), J19.2 (Pin_2), J20.1 (Pin_1), J21.1 (Pin_1), J22.1 (Pin_1), J23.1 (Pin_1), J8.5 (Pin_5), J9.5 (Pin_5)
- net at MOSFET5.3 (DRAIN): now also D7.2, J14.1 (Pin_1)
- net at J11.1 (Pin_1): now also MOSFET2.3 (DRAIN), D4.2; no longer MOSFET8.3 (DRAIN)
- net at U8.3 (SW), U8.8 (SW): now also D10.1, L1.2
- net at P1.2 (TCT), P1.5 (RCT): now also C15.2
- net at MOSFET6.3 (DRAIN): now also D8.2, J15.1 (Pin_1)
- net at MOSFET7.3 (DRAIN): now also D9.2, J16.1 (Pin_1)
- net at U8.11 (PWRGD): now also R5.1
- net at U8.13 (COMP): now also R6.1
- net at U8.19 (BIAS): now also C25.1, R7.1
- net at D1.2, J1.1: now also C6.2, R1.1
- net at D1.1, J1.2: now also C4.2, R2.1
- net V_USB_IN: no longer names the net of U4.49 (VUSB)
- new net: D12.2, J18.1 (Pin_1), MOSFET9.3 (DRAIN)
- new net: C27.2, R6.2
- new net: D11.2, J17.1 (Pin_1), MOSFET8.3 (DRAIN)
- new net: D13.2, J19.1 (Pin_1), MOSFET10.3 (DRAIN)
- new net SPI_1_MOSI: J6.3 (Pin_3)
- no-connect marks 0 -> 1
Other:
- note added: "Asked Asher about EECS caps"
- note added: "TBD RS485"
- note added: "Teensy Pinout"
- note removed: "Create Pinouts"
