File: Pneumatics Control Unit Pin (Senior Design)/Pneumatics Control Unit Pinned.kicad_sch (KiCad schematic)
At the start: 87 parts

Commit message: Senior Update
Parts:
- removed C16: (no value), symbol Samsung Cap 22u:CL21A226MQQNNNF
- removed C17, C25, C26, C28: (no value), symbol Device:C
- removed CR1: (no value), symbol MBRS130L Diode:MBRS130L
- removed D1, D2: (no value), symbol Device:D_TVS_x2_AAC
- removed J3: (no value), symbol USB 2.0 Micro:10118194-0001LF
- removed L1: (no value), symbol Taiyo Inductor 33uh:LB3218T330KV
- removed MOSFET1, MOSFET10, MOSFET2, MOSFET3, MOSFET4, MOSFET5, MOSFET6, MOSFET7, MOSFET8, MOSFET9: (no value), symbol Toshiba MOSFET:SSM3K7002KFU
- removed R5, R6, R7: (no value), symbol Device:R_US
- removed U7: (no value), symbol RS485 To UART:ISL83490IBZ
- removed U8: (no value), symbol 3.3Sw:MIC2178-3.3YWM
- added C?: CL21A226MQQNNNF, symbol Samsung Cap 22u:CL21A226MQQNNNF
- added C?: 0.1u, Capacitor_SMD:C_0805_2012Metric_Pad1.18x1.45mm_HandSolder, symbol Device:C
- added C?: 6.8n, Capacitor_SMD:C_0805_2012Metric_Pad1.18x1.45mm_HandSolder, symbol Device:C
- added C?: 0.01u, Capacitor_SMD:C_0805_2012Metric_Pad1.18x1.45mm_HandSolder, symbol Device:C
- added C?: 1u, Capacitor_SMD:C_0805_2012Metric_Pad1.18x1.45mm_HandSolder, symbol Device:C
- added CR?: MBRS130L, symbol MBRS130L Diode:MBRS130L
- added D?: PESD1FLEX,215, Dual Diode:PESD1FLEX215, symbol Dual Diode:PESD1FLEX,215
- added D?: (no value), Dual Diode:PESD1FLEX215, symbol Dual Diode:PESD1FLEX,215
- added J3: (no value), symbol USB 2.0 Type A:87583-2010BLF
- added L?: LB3218T330KV, symbol Taiyo Inductor 33uh:LB3218T330KV
- added MOSFET?: (no value), symbol Toshiba MOSFET:SSM3K7002KFU
- added MOSFET? (x9): SSM3K7002KFU, Toshiba MOSFET:SSM3K7002KFU, symbol Toshiba MOSFET:SSM3K7002KFU
- added R?: 20k, Resistor_SMD:R_0805_2012Metric_Pad1.20x1.40mm_HandSolder, symbol Device:R_US
- added R? (x2): 10k, Resistor_SMD:R_0805_2012Metric_Pad1.20x1.40mm_HandSolder, symbol Device:R_US
- added U?: (no value), symbol RS485 To UART:ISL83490IBZ
- added U?: (no value), symbol 33SW:MIC2178-3.3YWM
Connections:
- net 220uF: now also C?.1, L?.2, U?.12 (FB)
- net GND: now also C?.2, C?.2, C?.2, C?.2, C?.2, CR?.2, D?.3, D?.3, J3.1 (GND), MOSFET?.2 (SOURCE), MOSFET?.2 (SOURCE), MOSFET?.2 (SOURCE), MOSFET?.2 (SOURCE), MOSFET?.2 (SOURCE), MOSFET?.2 (SOURCE), MOSFET?.2 (SOURCE), MOSFET?.2 (SOURCE), MOSFET?.2 (SOURCE), MOSFET?.2 (SOURCE), R?.2, U?.10 (*PWM), U?.14 (SGND), U?.15 (SGND), U?.16 (SGND), U?.17 (SGND), U?.18 (SYNC), U?.4 (PGND), U?.5 (PGND), U?.6 (PGND), U?.7 (PGND)
- net GPIO_0: now also MOSFET?.1 (GATE)
- net GPIO_1: now also MOSFET?.1 (GATE)
- net GPIO_2: now also MOSFET?.1 (GATE)
- net GPIO_3: now also MOSFET?.1 (GATE)
- net GPIO_4: now also MOSFET?.1 (GATE)
- net GPIO_5: now also MOSFET?.1 (GATE)
- net GPIO_6: now also MOSFET?.1 (GATE)
- net GPIO_7: now also MOSFET?.1 (GATE)
- net GPIO_8: now also MOSFET?.1 (GATE)
- net GPIO_9: now also MOSFET?.1 (GATE)
- net RS485_A_12V: now also C?.1, C?.1, R?.2, U?.1 (VIN), U?.2 (VIN), U?.20 (EN), U?.9 (VIN)
- net RS485_RXD: now also U?.3 (DI)
- net RS485_TXD: now also U?.2 (RO)
- net USB_D+: now also J3.2 (D+)
- net USB_D-: now also J3.3 (D-)
- net at D5.2 (A2), J6.1 (Pin_1): now also MOSFET?.3 (DRAIN)
- net at D12.2 (A2), J13.1 (Pin_1): now also MOSFET?.3 (DRAIN)
- net at D11.2 (A2), J12.1 (Pin_1): now also MOSFET?.3 (DRAIN)
- net at D4.2 (A2), J5.1 (Pin_1): now also MOSFET?.3 (DRAIN)
- net at D10.2 (A2), J11.1 (Pin_1): now also MOSFET?.3 (DRAIN)
- net at C5.1, C7.1, J2.1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: now also D?.1, D?.2
- net at D3.2 (A2), J4.1 (Pin_1): now also MOSFET?.3 (DRAIN)
- net at D6.2 (A2), J7.1 (Pin_1): now also MOSFET?.3 (DRAIN)
- net at D7.2 (A2), J8.1 (Pin_1): now also MOSFET?.3 (DRAIN)
- net at R3.2: now also U?.6 (Z)
- net at D9.2 (A2), J10.1 (Pin_1): now also MOSFET?.3 (DRAIN)
- net at D8.2 (A2), J9.1 (Pin_1): now also MOSFET?.3 (DRAIN)
- net at C11.1, C12.1, C13.1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: now also J3.4 (VCC)
- net at C6.1, J1.1, R1.1: now also D?.2
- net at C4.1, J1.2: now also R2.2, D?.1; no longer R2.1
- net at R4.2: now also U?.5 (Y)
- net at R1.2: now also U?.8 (A)
- new net: R2.1, U?.7 (B)
- new net: CR?.1, L?.1, U?.3 (SW), U?.8 (SW)
- new net: C?.1, R?.2
- new net: R?.1, U?.11 (PWRGD)
- new net: R?.1, U?.13 (COMP)
- new net: C?.1, R?.1, U?.19 (BIAS)
Other:
- note added: "USB 2.0 Type A"
- note removed: "USB 2.0 Micro"
- moved on the sheet: C11, C12, C13, C14, R2, R4

Commit message: Senior update
Parts:
- removed C11, C12, C13, C14, C15, C4, C5, C6, C7: (no value), symbol Device:C
- removed D10, D11, D12, D3, D4, D5, D6, D7, D8, D9: (no value), symbol Device:D_TVS_x2_AAC
- removed J10, J11, J12, J13, J5, J6, J7, J8, J9: (no value), symbol Connector:Conn_01x02_Male
- added C? (x6): 0.1u, 0.1 uF Cap:0402YC104KAT2A, symbol 0.1 uF Cap:0402YC104KAT2A
- added C?: (no value), symbol 10 nF Cap:0402YC103KAT2A
- added C?: (no value), 10 nF Cap:0402YC103KAT2A, symbol 10 nF Cap:0402YC103KAT2A
- added C?: (no value), 0.1 uF Cap:0402YC104KAT2A, symbol 0.1 uF Cap:0402YC104KAT2A
- added D? (x10): PESD1FLEX,215, Dual Diode:PESD1FLEX215, symbol Dual Diode:PESD1FLEX,215
- added J? (x9): Conn_01x02_Male, Connector_PinSocket_2.54mm:PinSocket_1x02_P2.54mm_Vertical, symbol Connector:Conn_01x02_Male
- C1, C10, C2, C3, C8, C9: value (none) -> 1u; footprint (none) -> Capacitor_SMD:C_0805_2012Metric_Pad1.18x1.45mm_HandSolder
- C16: renamed from C?; footprint (none) -> Samsung-CL21-09_2016-0-*
- C18, C19, C20, C21, C22, C23, C24, C27, C29, C30: value (none) -> CL21A226MQQNNNF; footprint (none) -> Samsung-CL21-09_2016-0-*
- CR1: renamed from CR?; footprint (none) -> DIODE_DO214AA
- D1: renamed from D?; value (none) -> PESD1FLEX,215
- H1, H2, H3, H4: value (none) -> MountingHole; footprint (none) -> MountingHole:MountingHole_2.5mm
- J1: value (none) -> RX_PORT; footprint (none) -> RS485:RS485
- J2: value (none) -> TX_PORT; footprint (none) -> RS485:RS485
- J3: value (none) -> 87583-2010BLF; footprint (none) -> USB 2.0 Type A:87583-2010BLF
- J4: value (none) -> Conn_01x02_Male; footprint (none) -> Connector_PinSocket_2.54mm:PinSocket_1x02_P2.54mm_Vertical
- L1: renamed from L?; footprint (none) -> INDC3218X200N
- MOSFET1: renamed from MOSFET?; value (none) -> SSM3K7002KFU; footprint (none) -> Toshiba MOSFET:SSM3K7002KFU
- P1: value (none) -> J1B1211CCD; footprint (none) -> Ethernet:J1B1211CCD; Price None -> $3.78; Source (none) -> https://www.digikey.com/en/products/detail/wiznet/J1B1211CC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
- R1, R2, R3, R4: value (none) -> 10; footprint (none) -> Resistor_SMD:R_0805_2012Metric_Pad1.20x1.40mm_HandSolder
- U1, U2, U3: value (none) -> MC78M05CDTRKG; footprint (none) -> 12V5V Regulator:MC78M05CDTRKG; Price (none) -> $0.54; Source (none) -> https://www.digikey.com/en/products/detail/onsemi/MC78M05CD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
- U4: value (none) -> Teensy4.1; footprint (none) -> Teensy:Teensy41; Price (none) -> $26.85; Source (none) -> https://www.pjrc.com/store/teensy41.html
- U5, U6: value (none) -> 74AXP2T3407GSX; footprint (none) -> Nexperia Level Shifter:74AXP2T3407GSX
- U7: renamed from U?; footprint (none) -> RS485 To UART:ISL83490IBZ
- U8: renamed from U?; Price (none) -> $8.01; Source (none) -> https://www.digikey.com/en/products/detail/microchip-techno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
- gave numbers to parts that had none: 17
Connections:
- net 220uF is gone; now on net +3V3: C18.1, C19.1, C20.1, C21.1, C22.1, C23.1, C24.1, C27.1, C28.1, C29.1, C30.1, L1.2, U8.12 (FB)
- net GND: now also U7.4 (GND), C?.1, C?.1, C?.1, C?.1, C?.1, C?.1, C?.1, C?.1, C?.1, D?.3, D?.3, D?.3, D?.3, D?.3, D?.3, D?.3, D?.3, D?.3, D?.3; no longer U1.4 (GROUND), U2.4 (GROUND), U3.4 (GROUND)
- net GPIO_0: now also D?.1
- net GPIO_1: now also D?.1
- net GPIO_2: now also D?.1
- net GPIO_3: now also D?.1
- net GPIO_4: now also D?.1
- net GPIO_5: now also D?.1
- net GPIO_6: now also D?.1
- net GPIO_7: now also D?.1
- net GPIO_8: now also D?.1
- net GPIO_9: now also D?.1
- net RS485_B_12V: no longer U1.1 (INPUT), U2.1 (INPUT), U3.1 (INPUT)
- net at MOSFET10.3 (DRAIN): now also D?.2, J?.1 (Pin_1)
- net +3V3: now reaches U4.15 (3V3)
- net +3V3: now also U4.46 (3V3), U5.1 (VCCI), U6.1 (VCCI), U7.1 (VCC)
- net at MOSFET9.3 (DRAIN): now also D?.2, J?.1 (Pin_1)
- net at MOSFET3.3 (DRAIN): now also D?.2, J?.1 (Pin_1)
- net at D2.1, D2.2, J2.1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: now also C?.2, C?.2
- net at J4.1 (Pin_1), MOSFET1.3 (DRAIN): now also D?.2
- net at MOSFET4.3 (DRAIN): now also D?.2, J?.1 (Pin_1)
- net +5V: now reaches U5.8 (VCCO), U6.8 (VCCO)
- net +5V: now also C10.1, C8.1, C9.1, J3.4 (VCC), J4.2 (Pin_2), C?.2, C?.2, C?.2, C?.2, J?.2 (Pin_2), J?.2 (Pin_2), J?.2 (Pin_2), J?.2 (Pin_2), J?.2 (Pin_2), J?.2 (Pin_2), J?.2 (Pin_2), J?.2 (Pin_2), J?.2 (Pin_2)
- net at MOSFET5.3 (DRAIN): now also D?.2, J?.1 (Pin_1)
- net at MOSFET8.3 (DRAIN): now also D?.2, J?.1 (Pin_1)
- net at P1.2 (TCT), P1.5 (RCT): now also C?.2
- net at MOSFET6.3 (DRAIN): now also D?.2, J?.1 (Pin_1)
- net at MOSFET2.3 (DRAIN): now also D?.2, J?.1 (Pin_1)
- net at MOSFET7.3 (DRAIN): now also D?.2, J?.1 (Pin_1)
- net at D1.2, J1.1, R1.1: now also C?.2
- net at D1.1, J1.2, R2.2: now also C?.2
- now unconnected: U1.3 (OUTPUT), U2.3 (OUTPUT), U3.3 (OUTPUT)
Other:
- note added: "All Pneumatics complete"
- note added: "Asked Asher about EECS caps"
- moved on the sheet: U1, U2, U3

Commit message: Senior Update
Parts:
- removed C1, C10, C17, C2, C3, C8, C9: 1u, Capacitor_SMD:C_0805_2012Metric_Pad1.18x1.45mm_HandSolder, symbol Device:C
- removed C16, C18, C19, C20, C21, C22, C23, C24, C27, C29, C30: CL21A226MQQNNNF, Samsung-CL21-09_2016-0-*, symbol Samsung Cap 22u:CL21A226MQQNNNF
- removed C25: 0.01u, Capacitor_SMD:C_0805_2012Metric_Pad1.18x1.45mm_HandSolder, symbol Device:C
- removed C26: 6.8n, Capacitor_SMD:C_0805_2012Metric_Pad1.18x1.45mm_HandSolder, symbol Device:C
- removed C28: 0.1u, Capacitor_SMD:C_0805_2012Metric_Pad1.18x1.45mm_HandSolder, symbol Device:C
- removed CR1: MBRS130L, DIODE_DO214AA, symbol MBRS130L Diode:MBRS130L
- removed L1: LB3218T330KV, INDC3218X200N, symbol Taiyo Inductor 33uh:LB3218T330KV
- removed R5: 20k, Resistor_SMD:R_0805_2012Metric_Pad1.20x1.40mm_HandSolder, symbol Device:R_US
- removed R6, R7: 10k, Resistor_SMD:R_0805_2012Metric_Pad1.20x1.40mm_HandSolder, symbol Device:R_US
- removed U1, U2, U3: MC78M05CDTRKG, 12V5V Regulator:MC78M05CDTRKG, symbol 12V5V Regulator:MC78M05CDTRKG
- added C? (x7): (no value), 1 uF Cap:C1608X7R1C105K080AC, symbol 1 uF Cap:C1608X7R1C105K080AC
- added C? (x2): (no value), 22 uF Cap:CL21A226MQQNNNE, symbol 22 uF Cap:CL21A226MQQNNNE
- added C?: (no value), 6.8 nF Cap:0402B682K500CT, symbol 6.8 nF Cap:0402B682K500CT
- added C? (x9): 22u, 22 uF Cap:CL21A226MQQNNNE, symbol 22 uF Cap:CL21A226MQQNNNE
- added C?: (no value), 0.01 uF cap:CL05B103KO5NNNC, symbol 0.01 uF Cap:CL05B103KO5NNNC
- added C?: 0.1u, 0.1 uF Cap:0402YC104KAT2A, symbol 0.1 uF Cap:0402YC104KAT2A
- added D?: (no value), CDBA340-HF Diode:CDBA340-HF, symbol CDBA340-HF Diode:CDBA340-HF
- added L?: (no value), 33 uH Inductor:LB3218T330K, symbol 33 uH Inductor:LB3218T330K
- added R?: (no value), 20K Res:SR1-0805-320, symbol 20K Res:SR1-0805-320
- added R?: 10K, 10K Res:SR1-0603-310, symbol 10K Res:SR1-0603-310
- added R?: (no value), 10K Res:SR1-0603-310, symbol 10K Res:SR1-0603-310
- added U? (x2): MC78M05CDTRKG, 12V5V Regulator:MC78M05CDTRKG, symbol 12V5V Regulator:MC78M05CDTRKG
- added U?: (no value), symbol 12V5V Regulator:MC78M05CDTRKG
- C?: footprint (none) -> 10 nF Cap:0402YC103KAT2A
- U8: footprint (none) -> 33SW:MIC2178-33YWM
Connections:
- net V_IN is gone; now on net +5V: U4.48 (VIN)
- net +3V3: now also C?.2, C?.2, C?.2, C?.2, C?.2, C?.2, C?.2, C?.2, C?.2, C?.2, C?.2, L?.1
- net +5V: now also C?.2, C?.2, C?.2, U?.3 (OUTPUT), U?.3 (OUTPUT), U?.3 (OUTPUT)
- net GND: now also C?.1, C?.1, C?.1, C?.1, C?.1, C?.1, C?.1, C?.1, C?.1, C?.1, C?.1, C?.1, C?.1, C?.1, C?.1, C?.1, C?.1, C?.1, C?.1, C?.1, C?.2, D?.2, R?.2, U?.4 (GROUND), U?.4 (GROUND), U?.4 (GROUND)
- net RS485_A_12V: now also C?.2, C?.2, R?.2
- net RS485_B_12V: now also C?.2, C?.2, C?.2, U?.1 (INPUT), U?.1 (INPUT), U?.1 (INPUT)
- net at U8.3 (SW), U8.8 (SW): now also D?.1, L?.2
- net at U8.11 (PWRGD): now also R?.1
- net at U8.13 (COMP): now also R?.1
- net at U8.19 (BIAS): now also C?.1, R?.1
- net V_USB_IN: no longer names the net of U4.49 (VUSB)
- new net: C?.2, R?.2
- no-connect marks 0 -> 1
Other:
- note added: "Asked Asher about EECS caps TBD RS485"
- note added: "Might have to add Header Pins"

Commit message: Senior update
Parts:
- removed R1, R2, R3, R4: 10, Resistor_SMD:R_0805_2012Metric_Pad1.20x1.40mm_HandSolder, symbol Device:R_US
- added J10, J8, J9: (no value), symbol Connector:Conn_01x05_Male
- added J5: (no value), symbol Connector:Conn_01x12_Male
- added J6: (no value), symbol Connector:Conn_01x04_Male
- added J7: (no value), symbol Connector:Conn_01x10_Male
- added R1, R2, R3: 10, 10 Res:RNCP0603FTD10R0, symbol 10 Res:RNCP0603FTD10R0
- added R4: (no value), 10 Res:RNCP0603FTD10R0, symbol 10 Res:RNCP0603FTD10R0
- C1, C10, C17, C2, C3, C8, C9: renamed from C?; value (none) -> 1u
- C13, C14: renamed from C?; value (none) -> 10n
- C16, C30: renamed from C?; value (none) -> 22u
- C25: renamed from C?; value (none) -> 0.01u
- C27: renamed from C?; value (none) -> 6.8n
- C6: renamed from C?; value (none) -> 0.1u
- D10: renamed from D?; value (none) -> CDBA340-HF
- J1: value RX_PORT -> (none); footprint RS485:RS485 -> (none)
- L1: renamed from L?; value (none) -> 33u
- R5: renamed from R?; value (none) -> 20k
- R7: renamed from R?; value (none) -> 10K
- U1: renamed from U?; value (none) -> MC78M05CDTRKG; footprint (none) -> 12V5V Regulator:MC78M05CDTRKG
- U5, U6: Price (none) -> $0.64; Source (none) -> https://www.digikey.com/en/products/detail/nexperia-usa-inc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
- U7: value (none) -> ISL83490IBZ
- U8: value (none) -> MIC2178-3.3YWM
- gave numbers to parts that had none: 38
Connections:
- net +3V3: now also J10.4 (Pin_4), J8.4 (Pin_4), J9.4 (Pin_4)
- net +5V: now also J10.5 (Pin_5), J8.5 (Pin_5), J9.5 (Pin_5)
- net GND: now also J10.1 (Pin_1), J8.1 (Pin_1), J9.1 (Pin_1)
- net GPIO_10: now also J7.1 (Pin_1)
- net GPIO_11: now also J7.2 (Pin_2)
- net GPIO_12: now also J7.3 (Pin_3)
- net GPIO_13: now also J7.4 (Pin_4)
- net GPIO_14: now also J7.5 (Pin_5)
- net GPIO_15: now also J7.6 (Pin_6)
- net GPIO_16: now also J7.7 (Pin_7)
- net GPIO_17: now also J7.8 (Pin_8)
- net GPIO_18: now also J7.9 (Pin_9)
- net GPIO_19: now also J7.10 (Pin_10)
- net I2C_0_SCL: now also J8.2 (Pin_2)
- net I2C_0_SDA: now also J8.3 (Pin_3)
- net I2C_1_SCL: now also J9.3 (Pin_3)
- net I2C_1_SDA: now also J9.2 (Pin_2)
- net I2C_2_SCL: now also J10.3 (Pin_3)
- net I2C_2_SDA: now also J10.2 (Pin_2)
- net SPI_0_CS_0: now also J5.9 (Pin_9)
- net SPI_0_CS_1: now also J5.5 (Pin_5)
- net SPI_0_CS_2: now also J5.1 (Pin_1)
- net SPI_0_MISO: now also J5.10 (Pin_10), J5.2 (Pin_2), J5.6 (Pin_6)
- net SPI_0_MOSI: now also J5.11 (Pin_11), J5.3 (Pin_3), J5.7 (Pin_7)
- net SPI_0_SCK: now also J5.12 (Pin_12), J5.4 (Pin_4), J5.8 (Pin_8)
- net SPI_1_CS: now also J6.1 (Pin_1)
- net SPI_1_MISO: now also J6.2 (Pin_2)
- net SPI_1_SCK: now also J6.4 (Pin_4)
- net at U7.5 (Y): now also R4.2
- net at U7.6 (Z): now also R3.2
- net at U7.7 (B): now also R2.2
- net at U7.8 (A): now also R1.2
- net at C5.2, C7.2, D2.1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: now also R3.1, R4.1
- net at C4.2, D1.1, J1.2: now also R2.1
- net at C6.2, D1.2, J1.1: now also R1.1
- new net SPI_1_MOSI: J6.3 (Pin_3)
Other:
- note added: "TBD RS485"
- note added: "Teensy Pinout"
- note removed: "All Pneumatics complete"
- note removed: "Asked Asher about EECS caps TBD RS485"
- note removed: "Create Pinouts"
- note removed: "Might have to add Header Pins"

Commit message: Senior Update
Parts:
- added J20: Encoder 1 - CCW, symbol Connector:Conn_01x03_Female
- added J21, J23: (no value), symbol Connector:Conn_01x03_Female
- added J22: Encoder 1 - CW, symbol Connector:Conn_01x03_Female
- J1: value (none) -> RX_PORT; footprint (none) -> RS485:RS485
- J10: value (none) -> I2C 2
- J5: value (none) -> SPI 0
- J6: value (none) -> SPI 1
- J7: value (none) -> GPIO
- J8: value (none) -> I2C 0
- J9: value (none) -> I2C 1
- R4: value (none) -> 10
Connections:
- net +5V: now also J20.1 (Pin_1), J21.1 (Pin_1), J22.1 (Pin_1), J23.1 (Pin_1)
- net Encoder_0_CCW: now also J20.2 (Pin_2)
- net Encoder_0_CW: now also J22.2 (Pin_2)
- net Encoder_1_CCW: now also J21.2 (Pin_2)
- net Encoder_1_CW: now also J23.2 (Pin_2)
- net GND: now also J20.3 (Pin_3), J21.3 (Pin_3), J22.3 (Pin_3), J23.3 (Pin_3)

Commit message: Senior Update
Parts:
- J1: value RX_PORT -> (none); footprint RS485:RS485 -> (none); Price (none) -> $0.38; Source (none) -> https://www.digikey.com/en/products/detail/adam-tech/MTJ-64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
- J2: value TX_PORT -> (none); Price (none) -> $0.38; Source (none) -> https://www.digikey.com/en/products/detail/adam-tech/MTJ-64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
- J21: value (none) -> Encoder 2 - CCW
- J23: value (none) -> Encoder 2 - CW
Changed lines of the file:
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@@
       (effects (font (size 1.27 1.27)) (justify left))
     )
-    (property "Value" "" (id 1) (at 233.68 254 0)
+    (property "Value" "Encoder 2 - CW" (id 1) (at 233.68 254 0)
       (effects (font (size 1.27 1.27)) (justify left))
     )
@@
     (pin "2")
   )
+  (symbol (lib_id "Connector:4P4C") (at 25.4 59.69 0) (mirror x) (unit 1)
+    (in_bom yes) (on_board yes)
+    (property "Reference" "J2" (id 0) (at 25.4 72.39 0)
+      (effects (font (size 1.27 1.27)))
+    )
+    (property "Value" "" (id 1) (at 25.4 69.85 0)
+      (effects (font (size 1.27 1.27)))
+    )
+    (property "Footprint" "RS485:RS485" (id 2) (at 25.4 60.96 90)
+      (effects (font (size 1.27 1.27)) hide)
+    )
+    (property "Datasheet" "https://app.adam-tech.com/products/download/data_sheet/203851/mtj-642bx2-data-sheet.pdf" (id 3) (at 25.4 60.96 90)
+      (effects (font (size 1.27 1.27)) hide)
+    )
+    (property "Source" "https://www.digikey.com/en/products/detail/adam-tech/MTJ-642BX2/9832240" (id 4) (at 25.4 59.69 0)
+      (effects (font (size 1.27 1.27)) hide)
+    )
+    (property "Price" "$0.38" (id 5) (at 25.4 59.69 0)
+      (effects (font (size 1.27 1.27)) hide)
+    )
+    (pin "1")
+    (pin "2")
+    (pin "3")
+    (pin "4")
+  )
   (symbol (lib_id "power:GND") (at 111.76 275.59 0) (unit 1)
     (in_bom yes) (on_board yes)
@@
       (effects (font (size 1.27 1.27)) (justify left))
     )
-    (property "Value" "" (id 1) (at 209.55 255.27 0)
+    (property "Value" "Encoder 2 - CCW" (id 1) (at 209.55 255.27 0)
       (effects (font (size 1.27 1.27)) (justify left))
     )
@@
       (effects (font (size 1.27 1.27)))
     )
-    (property "Value" "RX_PORT" (id 1) (at 25.4 40.64 0)
-      (effects (font (size 1.27 1.27)))
-    )
-    (property "Footprint" "RS485:RS485" (id 2) (at 25.4 31.75 90)
-      (effects (font (size 1.27 1.27)) hide)
-    )
-    (property "Datasheet" "~" (id 3) (at 25.4 31.75 90)
+    (property "Value" "" (id 1) (at 25.4 40.64 0)
+      (effects (font (size 1.27 1.27)))
+    )
+    (property "Footprint" "" (id 2) (at 25.4 31.75 90)
+      (effects (font (size 1.27 1.27)) hide)
+    )
+    (property "Datasheet" "https://app.adam-tech.com/products/download/data_sheet/203851/mtj-642bx2-data-sheet.pdf" (id 3) (at 25.4 31.75 90)
+      (effects (font (size 1.27 1.27)) hide)
+    )
+    (property "Source" "https://www.digikey.com/en/products/detail/adam-tech/MTJ-642BX2/9832240" (id 4) (at 25.4 30.48 0)
+      (effects (font (size 1.27 1.27)) hide)
+    )
+    (property "Price" "$0.38" (id 5) (at 25.4 30.48 0)
       (effects (font (size 1.27 1.27)) hide)
     )
@@
     (pin "2")
   )
-  (symbol (lib_id "Connector:4P4C") (at 25.4 59.69 0) (mirror x) (unit 1)
-    (in_bom yes) (on_board yes)
-    (property "Reference" "J2" (id 0) (at 25.4 72.39 0)
-      (effects (font (size 1.27 1.27)))
-    )
-    (property "Value" "TX_PORT" (id 1) (at 25.4 69.85 0)
-      (effects (font (size 1.27 1.27)))
-    )
-    (property "Footprint" "RS485:RS485" (id 2) (at 25.4 60.96 90)
-      (effects (font (size 1.27 1.27)) hide)
-    )
-    (property "Datasheet" "~" (id 3) (at 25.4 60.96 90)
-      (effects (font (size 1.27 1.27)) hide)
-    )
-    (pin "1")
-    (pin "2")
-    (pin "3")
-    (pin "4")
-  )
   (symbol (lib_id "power:GND") (at 302.26 195.58 0) (unit 1)
     (in_bom yes) (on_board yes)
@@
       (reference "J1") (unit 1) (value "RX_PORT") (footprint "RS485:RS485")
     )
-    (path "/c552a028-a93e-4fbc-95ca-f9fd9f7655f2"
+    (path "/82cb8cb3-b005-4e19-a831-b4eef890bc5e"
       (reference "J2") (unit 1) (value "TX_PORT") (footprint "RS485:RS485")
     )
