File: Pneumatics Control Unit Pin (Senior Design)/Pneumatics Control Unit Pinned.kicad_sch (KiCad schematic)
At the start: 97 parts, among them J10 I2C 2, J11 Conn_01x02_Male, J12 Conn_01x02_Male, J13 Conn_01x02_Male, J14 Conn_01x02_Male, J15 Conn_01x02_Male, J16 Conn_01x02_Male, J17 Conn_01x02_Male, J18 Conn_01x02_Male, J19 Conn_01x02_Male, J20 Encoder 1 - CCW, J21 Encoder 2 - CCW, J22 Encoder 1 - CW, J23 Encoder 2 - CW, J3 87583-2010BLF, J4 Conn_01x02_Male, J5 SPI 0, J6 SPI 1, J7 GPIO, J8 I2C 0, J9 I2C 1, P1 J1B1211CCD, U1 MC78M05CDTRKG, U2 MC78M05CDTRKG, U3 MC78M05CDTRKG, U4 Teensy4.1, U5 74AXP2T3407GSX, U6 74AXP2T3407GSX, U7 ISL83490IBZ, U8 MIC2178-3.3YWM

Commit message: Senior Update
Parts:
- removed J10: I2C 2, symbol Connector:Conn_01x05_Male
- removed J20: Encoder 1 - CCW, symbol Connector:Conn_01x03_Female
- removed J21: Encoder 2 - CCW, symbol Connector:Conn_01x03_Female
- removed J22: Encoder 1 - CW, symbol Connector:Conn_01x03_Female
- removed J23: Encoder 2 - CW, symbol Connector:Conn_01x03_Female
- removed J5: SPI 0, symbol Connector:Conn_01x12_Male
- removed J6: SPI 1, symbol Connector:Conn_01x04_Male
- removed J7: GPIO, symbol Connector:Conn_01x10_Male
- removed J8: I2C 0, symbol Connector:Conn_01x05_Male
- removed J9: I2C 1, symbol Connector:Conn_01x05_Male
- removed U1: MC78M05CDTRKG, 12V5V Regulator:MC78M05CDTRKG, symbol 12V5V Regulator:MC78M05CDTRKG
- removed U4: Teensy4.1, Teensy:Teensy41, symbol Teensy:Teensy4.1
- removed U5: 74AXP2T3407GSX, Nexperia Level Shifter:74AXP2T3407GSX, symbol Nexperia Level Shifter:74AXP2T3407GSX
- removed U7: ISL83490IBZ, RS485 To UART:ISL83490IBZ, symbol RS485 To UART:ISL83490IBZ
- added J10: Encoder, Header:Conn_2x4, symbol Connector_Generic:Conn_02x04_Top_Bottom
- added J5: GPIO Bank 0, Header:Conn_2x7, symbol Connector_Generic:Conn_02x07_Top_Bottom
- added J6: SPI 0, Header:Conn_2x4, symbol Connector_Generic:Conn_02x04_Top_Bottom
- added J7: Solenoid Power Selector, Header:Conn_1x3, symbol Connector:Conn_01x03_Male
- added J8: GPIO Bank 1, Header:Conn_2x9, symbol Connector_Generic:Conn_02x09_Top_Bottom
- added J9: I2C 1-2, Header:Conn_2x5, symbol Connector_Generic:Conn_02x05_Top_Bottom
- added U1: Teensy4.1, Teensy:Teensy41, symbol Teensy:Teensy4.1
- added U4: MC78M05CDTRKG, 12V5V Regulator:MC78M05CDTRKG, symbol 12V5V Regulator:MC78M05CDTRKG
- added U5: ISL83490IBZ, RS485 To UART:ISL83490IBZ, symbol RS485 To UART:ISL83490IBZ
- added U7: 74AXP2T3407GSX, Nexperia Level Shifter:74AXP2T3407GSX, symbol Nexperia Level Shifter:74AXP2T3407GSX
- C6: value 0.1u -> (none); footprint 0.1 uF Cap:0402YC104KAT2A -> (none)
- J1: value (none) -> RX_PORT; footprint (none) -> RS485:MTJ-642BX2
- J11, J12, J13, J14, J15, J16, J17, J18, J19, J4: footprint Connector_PinSocket_2.54mm:PinSocket_1x02_P2.54mm_Vertical -> Header:Conn_1x2
- J2: value (none) -> TX_PORT; footprint RS485:RS485 -> RS485:MTJ-642BX2
Connections:
- net +3V3: now also J5.2 (Pin_2), J5.9 (Pin_9), J8.11 (Pin_11), J8.2 (Pin_2), J9.2 (Pin_2), J9.7 (Pin_7), U5.1 (VCC), U7.1 (VCCI)
- net +5V: now also J10.1 (Pin_1), J10.5 (Pin_5), J5.1 (Pin_1), J5.8 (Pin_8), J7.1 (Pin_1), J8.1 (Pin_1), J8.10 (Pin_10), J9.1 (Pin_1), J9.6 (Pin_6), U1.48 (VIN), U4.3 (OUTPUT), U7.8 (VCCO); no longer J11.2 (Pin_2), J12.2 (Pin_2), J13.2 (Pin_2), J14.2 (Pin_2), J15.2 (Pin_2), J16.2 (Pin_2), J17.2 (Pin_2), J18.2 (Pin_2), J19.2 (Pin_2), J4.2 (Pin_2)
- net Encoder_0_CCW: now also U6.3 (2A), J10.7 (Pin_7)
- net Encoder_0_CW: now also U6.2 (1A), J10.6 (Pin_6)
- net Encoder_1_CCW: now also J10.3 (Pin_3), U7.2 (1A); no longer U6.2 (1A)
- net Encoder_1_CW: now also J10.2 (Pin_2), U7.3 (2A); no longer U6.3 (2A)
- net GND: now also J10.4 (Pin_4), J10.8 (Pin_8), J5.5 (Pin_5), J5.6 (Pin_6), J5.7 (Pin_7), J8.12 (Pin_12), J8.13 (Pin_13), J8.3 (Pin_3), J8.4 (Pin_4), J9.10 (Pin_10), J9.5 (Pin_5), U1.1 (GND), U1.34 (GND), U1.47 (GND), U1.50 (VBAT), U1.51 (3V3), U1.52 (GND), U1.53 (PROGRAM), U1.54 (ON_OFF), U1.58 (GND), U1.59 (GND), U1.64 (GND), U4.4 (GROUND), U5.4 (GND), U7.4 (GND), U7.5 (GND)
- net GPIO_0: now also U1.4 (2_OUT2)
- net GPIO_1: now also U1.5 (3_LRCLK2)
- net GPIO_10: now also J5.10 (Pin_10), U1.24 (32_OUT1B)
- net GPIO_11: now also J8.14 (Pin_14), U1.37 (15_A1_RX3_SPDIF_IN)
- net GPIO_12: now also J8.15 (Pin_15), U1.36 (14_A0_TX3_SPDIF_OUT)
- net GPIO_13: now also J8.16 (Pin_16), U1.33 (41_A17)
- net GPIO_14: now also J8.17 (Pin_17), U1.32 (40_A16)
- net GPIO_15: now also J8.18 (Pin_18), U1.31 (39_MISO1_OUT1A)
- net GPIO_16: now also J8.5 (Pin_5), U1.30 (38_CS1_IN1)
- net GPIO_17: now also J8.6 (Pin_6), U1.28 (36_CS)
- net GPIO_18: now also J8.7 (Pin_7), U1.27 (35_TX8)
- net GPIO_19: now also J8.8 (Pin_8), U1.26 (34_RX8)
- net GPIO_2: now also U1.6 (4_BCLK2)
- net GPIO_3: now also U1.7 (5_IN2)
- net GPIO_4: now also U1.8 (6_OUT1D)
- net GPIO_5: now also U1.11 (9_OUT1C)
- net GPIO_6: now also U1.20 (28_RX7)
- net GPIO_7: now also U1.21 (29_TX7)
- net GPIO_8: now also U1.22 (30_CRX3)
- net GPIO_9: now also U1.23 (31_CTX3)
- net I2C_0_SCL: now also J9.4 (Pin_4), U1.41 (19_A5_SCL)
- net I2C_0_SDA: now also J9.3 (Pin_3), U1.40 (18_A4_SDA)
- net I2C_1_SCL: now also J9.8 (Pin_8), U1.38 (16_A2_RX4_SCL1)
- net I2C_1_SDA: now also J9.9 (Pin_9), U1.39 (17_A3_TX4_SDA1)
- net I2C_2_SCL: now also J5.3 (Pin_3), U1.16 (24_A10_TX6_SCL2)
- net I2C_2_SDA: now also J5.4 (Pin_4), U1.17 (25_A11_RX6_SDA2)
- net LED_Ethernet: now also U1.61 (LED)
- net R+_Ethernet: now also U1.60 (R+)
- net R-_Ethernet: now also U1.65 (R-)
- net RS485_B_12V: now also J7.3 (Pin_3), U4.1 (INPUT)
- net RS485_RXD: now also U1.10 (8_TX2_IN1), U5.3 (DI)
- net RS485_TXD: now also U1.9 (7_RX2_OUT1A), U5.2 (RO)
- net SPI_0_CS_0: now also J6.4 (Pin_4), U1.12 (10_CS_MQSR)
- net SPI_0_CS_1: now also J6.8 (Pin_8), U1.29 (37_CS)
- net SPI_0_MISO: now also J6.3 (Pin_3), J6.7 (Pin_7), U1.14 (12_MISO_MQSL)
- net SPI_0_MOSI: now also J6.2 (Pin_2), J6.6 (Pin_6), U1.13 (11_MOSI_CTX1)
- net SPI_0_SCK: now also J6.1 (Pin_1), J6.5 (Pin_5), U1.35 (13_SCK_LED)
- net SPI_1_CS: now also J5.11 (Pin_11), U1.2 (0_RX1_CRX2_CS1)
- net SPI_1_MISO: now also J5.12 (Pin_12), U1.18 (26_A12_MOSI1), U1.3 (1_TX1_CTX2_MISO1)
- net SPI_1_MOSI: now also J5.13 (Pin_13)
- net SPI_1_SCK: now also J5.14 (Pin_14), U1.19 (27_A13_SCK1)
- net T+_Ethernet: now also U1.63 (T+)
- net T-_Ethernet: now also U1.62 (T-)
- net USB_D+: now also U1.57 (D+)
- net USB_D-: now also U1.56 (D-)
- net USB_IN_D+: now also U1.67 (D+)
- net USB_IN_D-: now also U1.66 (D-)
- net V_USB: now also U1.55 (5V)
- net at C5.2, D2.1, J2.2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: no longer C7.2, D2.2, J2.1, R3.1
- net at R4.2: now also U5.5 (Y)
- net at R1.2: now also U5.8 (A)
- net at U6.7 (1Y): now also U1.45 (23_A9_CRX1_MCLK1)
- net at U6.6 (2Y): now also U1.44 (22_A8_CTX1)
- net at R3.2: now also U5.6 (Z)
- net at R2.2: now also U5.7 (B)
- new net: C7.2, D2.2, J2.1, R3.1
- new net: U1.43 (21_A7_RX5_BCLK1), U7.6 (2Y)
- new net: U1.42 (20_A6_TX5_LRCLK1), U7.7 (1Y)
- new net GPIO_20: J8.9 (Pin_9), U1.25 (33_MCLK2)
- new net Solenoid_Power: J11.2 (Pin_2), J12.2 (Pin_2), J13.2 (Pin_2), J14.2 (Pin_2), J15.2 (Pin_2), J16.2 (Pin_2), J17.2 (Pin_2), J18.2 (Pin_2), J19.2 (Pin_2), J4.2 (Pin_2), J7.2 (Pin_2)
- no-connect marks 1 -> 3
Other:
- note added: "Teensy Pinout $1.40 for 2x25 Header Male"
- note removed: "TBD RS485"
- note removed: "Teensy Pinout"

Commit message: Initial wiring, adding another 5V regulator for the GPIO pins, renumbered the mosfets
Parts:
- added U: (no value), symbol 12V5V Regulator:MC78M05CDTRKG
- added U (x2): (no value), symbol 1 uF Cap:C1608X7R1C105K080AC
- U: renamed from C13; value 10n -> (none); footprint 10 nF Cap:0402YC103KAT2A -> (none)
- U: renamed from C18; value 22u -> (none); footprint 22 uF Cap:CL21A226MQQNNNE -> (none)
- U: renamed from D4; value PESD1FLEX,215 -> (none); footprint Dual Diode:PESD1FLEX215 -> (none)
- U: renamed from D12; value PESD1FLEX,215 -> (none); footprint Dual Diode:PESD1FLEX215 -> (none)
- U: renamed from R1; value 10 -> (none); footprint 10 Res:RNCP0603FTD10R0 -> (none)
- U: renamed from MOSFET1; value SSM3K7002KFU -> (none); footprint Toshiba MOSFET:SSM3K7002KFU -> (none)
- U: renamed from MOSFET5; value SSM3K7002KFU -> (none); footprint Toshiba MOSFET:SSM3K7002KFU -> (none)
- U: renamed from J19; value Conn_01x02_Male -> (none); footprint Header:Conn_1x2 -> (none)
- U: renamed from C1; value 1u -> (none); footprint 1 uF Cap:C1608X7R1C105K080AC -> (none)
- U: renamed from C24; value 22u -> (none); footprint 22 uF Cap:CL21A226MQQNNNE -> (none)
- U: renamed from J6; value SPI 0 -> (none); footprint Header:Conn_2x4 -> (none)
- U: renamed from J11; value Conn_01x02_Male -> (none); footprint Header:Conn_1x2 -> (none)
- U: renamed from D7; value PESD1FLEX,215 -> (none); footprint Dual Diode:PESD1FLEX215 -> (none)
- U: renamed from C17; value 1u -> (none); footprint 1 uF Cap:C1608X7R1C105K080AC -> (none)
- U: renamed from J12; value Conn_01x02_Male -> (none); footprint Header:Conn_1x2 -> (none)
- U: renamed from R4; value 10 -> (none); footprint 10 Res:RNCP0603FTD10R0 -> (none)
- U: renamed from U6; value 74AXP2T3407GSX -> (none); footprint Nexperia Level Shifter:74AXP2T3407GSX -> (none)
- U: renamed from H2; value MountingHole -> (none); footprint MountingHole:MountingHole_2.5mm -> (none)
- U: renamed from C27; value 6.8n -> (none); footprint 6.8 nF Cap:0402B682K500CT -> (none)
- U: renamed from C7; value 0.1u -> (none); footprint 0.1 uF Cap:0402YC104KAT2A -> (none)
- U: renamed from MOSFET10; value SSM3K7002KFU -> (none); footprint Toshiba MOSFET:SSM3K7002KFU -> (none)
- U: renamed from C5; value 0.1u -> (none); footprint 0.1 uF Cap:0402YC104KAT2A -> (none)
- U: renamed from J7; value Solenoid Power Selector -> (none); footprint Header:Conn_1x3 -> (none)
- U: renamed from D8; value PESD1FLEX,215 -> (none); footprint Dual Diode:PESD1FLEX215 -> (none)
- U: renamed from C8; value 1u -> (none); footprint 1 uF Cap:C1608X7R1C105K080AC -> (none)
- U: renamed from H3; value MountingHole -> (none); footprint MountingHole:MountingHole_2.5mm -> (none)
- U: renamed from J13; value Conn_01x02_Male -> (none); footprint Header:Conn_1x2 -> (none)
- U: renamed from C20; value 22u -> (none); footprint 22 uF Cap:CL21A226MQQNNNE -> (none)
- U: renamed from D9; value PESD1FLEX,215 -> (none); footprint Dual Diode:PESD1FLEX215 -> (none)
- U: renamed from MOSFET9; value SSM3K7002KFU -> (none); footprint Toshiba MOSFET:SSM3K7002KFU -> (none)
- U: renamed from U7; value 74AXP2T3407GSX -> (none); footprint Nexperia Level Shifter:74AXP2T3407GSX -> (none)
- U: renamed from C11; value 0.1u -> (none); footprint 0.1 uF Cap:0402YC104KAT2A -> (none)
- U: renamed from C30; value 22u -> (none); footprint 22 uF Cap:CL21A226MQQNNNE -> (none)
- U: renamed from C4; value 0.1u -> (none); footprint 0.1 uF Cap:0402YC104KAT2A -> (none)
- U: renamed from J8; value GPIO Bank 1 -> (none); footprint Header:Conn_2x9 -> (none)
- U: renamed from R5; value 20k -> (none); footprint 20K Res:SR1-0805-320 -> (none)
- U: renamed from C21; value 22u -> (none); footprint 22 uF Cap:CL21A226MQQNNNE -> (none)
- U: renamed from D3; value PESD1FLEX,215 -> (none); footprint Dual Diode:PESD1FLEX215 -> (none)
- U: renamed from C15; value 0.1u -> (none); footprint 0.1 uF Cap:0402YC104KAT2A -> (none)
- U: renamed from L1; value 33u -> (none); footprint 33 uH Inductor:LB3218T330K -> (none)
- U: renamed from C16; value 22u -> (none); footprint 22 uF Cap:CL21A226MQQNNNE -> (none)
- U: renamed from C29; value 22u -> (none); footprint 22 uF Cap:CL21A226MQQNNNE -> (none)
- U: renamed from J9; value I2C 1-2 -> (none); footprint Header:Conn_2x5 -> (none)
- U: renamed from J17; value Conn_01x02_Male -> (none); footprint Header:Conn_1x2 -> (none)
- U: renamed from C12; value 0.1u -> (none); footprint 0.1 uF Cap:0402YC104KAT2A -> (none)
- U: renamed from H1; value MountingHole -> (none); footprint MountingHole:MountingHole_2.5mm -> (none)
- U: renamed from R2; value 10 -> (none); footprint 10 Res:RNCP0603FTD10R0 -> (none)
- U: renamed from H4; value MountingHole -> (none); footprint MountingHole:MountingHole_2.5mm -> (none)
- U: renamed from U1; value Teensy4.1 -> (none); footprint Teensy:Teensy41 -> (none)
- U: renamed from MOSFET4; value SSM3K7002KFU -> (none); footprint Toshiba MOSFET:SSM3K7002KFU -> (none)
- U: renamed from C25; value 0.01u -> (none); footprint 0.01 uF cap:CL05B103KO5NNNC -> (none)
- U: renamed from D13; value PESD1FLEX,215 -> (none); footprint Dual Diode:PESD1FLEX215 -> (none)
- U: renamed from MOSFET3; value SSM3K7002KFU -> (none); footprint Toshiba MOSFET:SSM3K7002KFU -> (none)
- U: renamed from C22; value 22u -> (none); footprint 22 uF Cap:CL21A226MQQNNNE -> (none)
- U: renamed from J16; value Conn_01x02_Male -> (none); footprint Header:Conn_1x2 -> (none)
- U: renamed from C26; value 22u -> (none); footprint 22 uF Cap:CL21A226MQQNNNE -> (none)
- U: renamed from C9; value 1u -> (none); footprint 1 uF Cap:C1608X7R1C105K080AC -> (none)
- U: renamed from C23; value 22u -> (none); footprint 22 uF Cap:CL21A226MQQNNNE -> (none)
- U: renamed from D6; value PESD1FLEX,215 -> (none); footprint Dual Diode:PESD1FLEX215 -> (none)
- U: renamed from R3; value 10 -> (none); footprint 10 Res:RNCP0603FTD10R0 -> (none)
- U: renamed from U8; value MIC2178-3.3YWM -> (none); footprint 33SW:MIC2178-33YWM -> (none)
- U: renamed from MOSFET6; value SSM3K7002KFU -> (none); footprint Toshiba MOSFET:SSM3K7002KFU -> (none)
- U: renamed from D11; value PESD1FLEX,215 -> (none); footprint Dual Diode:PESD1FLEX215 -> (none)
- U: renamed from C3; value 1u -> (none); footprint 1 uF Cap:C1608X7R1C105K080AC -> (none)
- U: renamed from C2; value 1u -> (none); footprint 1 uF Cap:C1608X7R1C105K080AC -> (none)
- U: renamed from J5; value GPIO Bank 0 -> (none); footprint Header:Conn_2x7 -> (none)
- U: renamed from MOSFET8; value SSM3K7002KFU -> (none); footprint Toshiba MOSFET:SSM3K7002KFU -> (none)
- U: renamed from J2; value TX_PORT -> (none); footprint RS485:MTJ-642BX2 -> (none)
- U: renamed from J18; value Conn_01x02_Male -> (none); footprint Header:Conn_1x2 -> (none)
- U: renamed from D1; value PESD1FLEX,215 -> (none); footprint Dual Diode:PESD1FLEX215 -> (none)
- U: renamed from J1; value RX_PORT -> (none); footprint RS485:MTJ-642BX2 -> (none)
- U: renamed from J15; value Conn_01x02_Male -> (none); footprint Header:Conn_1x2 -> (none)
- U: renamed from C14; value 10n -> (none); footprint 10 nF Cap:0402YC103KAT2A -> (none)
- U: renamed from D2; value PESD1FLEX,215 -> (none); footprint Dual Diode:PESD1FLEX215 -> (none)
- U: renamed from U2; value MC78M05CDTRKG -> (none); footprint 12V5V Regulator:MC78M05CDTRKG -> (none)
- U: renamed from C10; value 1u -> (none); footprint 1 uF Cap:C1608X7R1C105K080AC -> (none)
- U: renamed from U4; value MC78M05CDTRKG -> (none); footprint 12V5V Regulator:MC78M05CDTRKG -> (none)
- U: renamed from MOSFET7; value SSM3K7002KFU -> (none); footprint Toshiba MOSFET:SSM3K7002KFU -> (none)
- U: renamed from C19; value 22u -> (none); footprint 22 uF Cap:CL21A226MQQNNNE -> (none)
- U: renamed from R6; value 10K -> (none); footprint 10K Res:SR1-0603-310 -> (none)
- U: renamed from U5; value ISL83490IBZ -> (none); footprint RS485 To UART:ISL83490IBZ -> (none)
- U: renamed from U3; value MC78M05CDTRKG -> (none); footprint 12V5V Regulator:MC78M05CDTRKG -> (none)
- U: renamed from J3; value 87583-2010BLF -> (none); footprint USB 2.0 Type A:87583-2010BLF -> (none)
- U: renamed from J4; value Conn_01x02_Male -> (none); footprint Header:Conn_1x2 -> (none)
- U: renamed from R7; value 10K -> (none); footprint 10K Res:SR1-0603-310 -> (none)
- U: renamed from C28; value 0.1u -> (none); footprint 0.1 uF Cap:0402YC104KAT2A -> (none)
- U: renamed from P1; value J1B1211CCD -> (none); footprint Ethernet:J1B1211CCD -> (none)
- U: renamed from J10; value Encoder -> (none); footprint Header:Conn_2x4 -> (none)
- U: renamed from MOSFET2; value SSM3K7002KFU -> (none); footprint Toshiba MOSFET:SSM3K7002KFU -> (none)
- U: renamed from D10; value CDBA340-HF -> (none); footprint CDBA340-HF Diode:CDBA340-HF -> (none)
- U: renamed from D5; value PESD1FLEX,215 -> (none); footprint Dual Diode:PESD1FLEX215 -> (none)
- U: renamed from J14; value Conn_01x02_Male -> (none); footprint Header:Conn_1x2 -> (none)
- renumbered C6 to U
Connections:
- net +5V: now also U.2, U.3 (OUTPUT)
- net GND: now also U.1, U.1, U.4 (GROUND)
- net RS485_B_12V: now also U.1 (INPUT), U.2
- net SPI_1_MISO renamed SPI_1_MISO1
- net SPI_1_MISO1: no longer U.18 (26_A12_MOSI1)
- net SPI_1_MOSI renamed SPI_1_MOSI1
- net SPI_1_MOSI1: now also U.18 (26_A12_MOSI1)
Other:
- note added: "Pneumatics Power Rail -------------- 5v @ 0.5A -------------- Pneumatics: 0.1A x10 Teensy: ~0.1A - 0.35A NavX2 Micro: 0.05A Shaft Encoder: ~0.005A x2 External Pins: ~0.5A -------------- Total: ~1.91A"
- note removed: "Pneumatics Power Rail -------------- 5v @ 0.5A -------------- Pneumatics: 0.1A x10 Teensy: ~0.1A - 0.35A NavX2 Micro: 0.05A Shaft Encoder: ~0.005A x2 -------------- Total: ~1.41A"
- moved on the sheet: U
