File: Pneumatics Control Unit Pin (Senior Design)/Pneumatics Control Unit Pinned.kicad_sch (KiCad schematic)
At the start: 96 parts

Commit message: Adding labels for pinouts
Connections:
- net SPI_0_CS_0: no longer U.4 (Pin_4)
- net SPI_0_CS_1: no longer U.8 (Pin_8)
- new net SPI_0_CS: U.4 (Pin_4), U.8 (Pin_8)
Changed lines of the file:
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@@
     (effects (font (size 1.27 1.27)) (justify right bottom))
   )
-  (label "SPI_0_CS_0" (at 147.447 277.749 0) (fields_autoplaced)
+  (label "SPI_0_CS" (at 147.447 277.749 0) (fields_autoplaced)
     (effects (font (size 1.27 1.27)) (justify right bottom))
   )
@@
     (effects (font (size 1.27 1.27)) (justify left bottom))
   )
-  (label "SPI_0_CS_1" (at 165.227 277.749 0) (fields_autoplaced)
+  (label "SPI_0_CS" (at 165.227 277.749 0) (fields_autoplaced)
     (effects (font (size 1.27 1.27)) (justify left bottom))
   )
@@
   )
   (symbol_instances
+    (path "/a96442ef-a567-43e7-bb2f-3d8cc3d38530"
+      (reference "#PWR00") (unit 1) (value "GND") (footprint "")
+    )
     (path "/e6fc3c4d-354d-4397-bcf9-2ff452adbf52"
       (reference "#PWR0101") (unit 1) (value "GND") (footprint "")
@@
       (reference "#PWR0178") (unit 1) (value "GND") (footprint "")
     )
-    (path "/a96442ef-a567-43e7-bb2f-3d8cc3d38530"
-      (reference "#PWR?") (unit 1) (value "GND") (footprint "")
+    (path "/f0b593dc-4dfa-44bc-b395-79988370594d"
+      (reference "C0") (unit 1) (value "1u") (footprint "1 uF Cap:C1608X7R1C105K080AC")
     )
     (path "/19ddc83e-fdbf-4854-b635-0a005a96e472"
@@
     )
     (path "/ea4cfbc2-db63-4b8d-9630-af085d212d23"
-      (reference "C?") (unit 1) (value "1u") (footprint "1 uF Cap:C1608X7R1C105K080AC")
-    )
-    (path "/f0b593dc-4dfa-44bc-b395-79988370594d"
-      (reference "C?") (unit 1) (value "1u") (footprint "1 uF Cap:C1608X7R1C105K080AC")
+      (reference "C31") (unit 1) (value "1u") (footprint "1 uF Cap:C1608X7R1C105K080AC")
     )
     (path "/d33a4736-c811-4d0c-a054-0d71b90aa4de"
@@
       (reference "R7") (unit 1) (value "10K") (footprint "10K Res:SR1-0603-310")
     )
+    (path "/dbefbbf9-de0e-42bd-982e-9ca5f987f5b6"
+      (reference "U0") (unit 1) (value "MC78M05CDTRKG") (footprint "12V5V Regulator:MC78M05CDTRKG")
+    )
     (path "/83fcacc7-e5aa-4a4b-bdc7-bc44cd7f6326"
       (reference "U1") (unit 1) (value "Teensy4.1") (footprint "Teensy:Teensy41")
@@
       (reference "U8") (unit 1) (value "MIC2178-3.3YWM") (footprint "33SW:MIC2178-33YWM")
     )
-    (path "/dbefbbf9-de0e-42bd-982e-9ca5f987f5b6"
-      (reference "U?") (unit 1) (value "MC78M05CDTRKG") (footprint "12V5V Regulator:MC78M05CDTRKG")
-    )
   )
