File: Pneumatics Control Unit Pin (Senior Design)/Pneumatics Control Unit Pinned.kicad_pcb (KiCad board)
At the start: 0 parts

Commit message: Senior Update
Parts:
- added C1: 1u, 1 uF Cap:C1608X7R1C105K080AC, F.Cu at (38.0, 48.3)
- added C10: 1u, 1 uF Cap:C1608X7R1C105K080AC, F.Cu at (59.9, 25.1)
- added C11: 0.1u, 0.1 uF Cap:0402YC104KAT2A, F.Cu at (186.5, 99.8)
- added C12: 0.1u, 0.1 uF Cap:0402YC104KAT2A, F.Cu at (186.5, 106.7)
- added C13: 10n, 10 nF Cap:0402YC103KAT2A, F.Cu at (193.3, 91.9)
- added C14: 10n, 10 nF Cap:0402YC103KAT2A, F.Cu at (201.7, 94.5)
- added C15: 0.1u, 0.1 uF Cap:0402YC104KAT2A, F.Cu at (53.3, 91.4)
- added C16: 22u, 22 uF Cap:CL21A226MQQNNNE, F.Cu at (102.1, 75.2)
- added C17: 1u, 1 uF Cap:C1608X7R1C105K080AC, F.Cu at (101.6, 83.3)
- added C18: 22u, 22 uF Cap:CL21A226MQQNNNE, F.Cu at (135.2, 75.9)
- added C19: 22u, 22 uF Cap:CL21A226MQQNNNE, F.Cu at (125.7, 80.7)
- added C2: 1u, 1 uF Cap:C1608X7R1C105K080AC, F.Cu at (38.0, 45.7)
- added C20: 22u, 22 uF Cap:CL21A226MQQNNNE, F.Cu at (120.0, 96.8)
- added C21: 22u, 22 uF Cap:CL21A226MQQNNNE, F.Cu at (114.5, 91.9)
- added C22: 22u, 22 uF Cap:CL21A226MQQNNNE, F.Cu at (130.2, 87.6)
- added C23: 22u, 22 uF Cap:CL21A226MQQNNNE, F.Cu at (133.3, 70.0)
- added C24: 22u, 22 uF Cap:CL21A226MQQNNNE, F.Cu at (117.9, 74.6)
- added C25: 0.01u, 0.01 uF cap:CL05B103KO5NNNC, F.Cu at (105.2, 77.7)
- added C26: 22u, 22 uF Cap:CL21A226MQQNNNE, F.Cu at (117.9, 82.8)
- added C27: 6.8n, 6.8 nF Cap:0402B682K500CT, F.Cu at (106.2, 74.7)
- added C28: 0.1u, 0.1 uF Cap:0402YC104KAT2A, F.Cu at (97.5, 77.7)
- added C29: 22u, 22 uF Cap:CL21A226MQQNNNE, F.Cu at (125.1, 74.6)
- added C3: 1u, 1 uF Cap:C1608X7R1C105K080AC, F.Cu at (38.0, 43.2)
- added C30: 22u, 22 uF Cap:CL21A226MQQNNNE, F.Cu at (122.9, 87.6)
- added C4: 0.1u, 0.1 uF Cap:0402YC104KAT2A, F.Cu at (44.8, 67.6)
- added C5: 0.1u, 0.1 uF Cap:0402YC104KAT2A, F.Cu at (44.8, 50.3)
- added C6: 0.1u, 0.1 uF Cap:0402YC104KAT2A, F.Cu at (44.8, 76.7)
- added C7: 0.1u, 0.1 uF Cap:0402YC104KAT2A, F.Cu at (44.8, 59.4)
- added C8: 1u, 1 uF Cap:C1608X7R1C105K080AC, F.Cu at (62.0, 25.1)
- added C9: 1u, 1 uF Cap:C1608X7R1C105K080AC, F.Cu at (64.0, 25.1)
- added D1: PESD1FLEX,215, Dual Diode:PESD1FLEX215, F.Cu at (45.8, 72.1)
- added D10: CDBA340-HF, CDBA340-HF Diode:CDBA340-HF, F.Cu at (89.5, 80.8)
- added D11: PESD1FLEX,215, Dual Diode:PESD1FLEX215, F.Cu at (-34.7, 10.5)
- added D12: PESD1FLEX,215, Dual Diode:PESD1FLEX215, F.Cu at (-41.0, 48.6)
- added D13: PESD1FLEX,215, Dual Diode:PESD1FLEX215, F.Cu at (-35.1, 85.3)
- added D2: PESD1FLEX,215, Dual Diode:PESD1FLEX215, F.Cu at (45.8, 54.9)
- added D3: PESD1FLEX,215, Dual Diode:PESD1FLEX215, F.Cu at (-121.8, 12.1)
- added D4: PESD1FLEX,215, Dual Diode:PESD1FLEX215, F.Cu at (-115.9, 46.6)
- added D5: PESD1FLEX,215, Dual Diode:PESD1FLEX215, F.Cu at (-112.0, 84.3)
- added D6: PESD1FLEX,215, Dual Diode:PESD1FLEX215, F.Cu at (-108.8, 112.1)
- added D7: PESD1FLEX,215, Dual Diode:PESD1FLEX215, F.Cu at (-80.3, 13.2)
- added D8: PESD1FLEX,215, Dual Diode:PESD1FLEX215, F.Cu at (-75.0, 47.8)
- added D9: PESD1FLEX,215, Dual Diode:PESD1FLEX215, F.Cu at (-67.8, 89.7)
- added G***: LOGO, look of disapproval:look of disapproval, F.Cu at (58.8, 33.8)
- added H1: MountingHole, MountingHole:MountingHole_2.5mm, F.Cu at (266.7, 129.5)
- added H2: MountingHole, MountingHole:MountingHole_2.5mm, F.Cu at (274.3, 145.3)
- added H3: MountingHole, MountingHole:MountingHole_2.5mm, F.Cu at (271.8, 157.0)
- added H4: MountingHole, MountingHole:MountingHole_2.5mm, F.Cu at (259.6, 138.9)
- added J1: RX_PORT, RS485:MTJ-642BX2, F.Cu at (33.6, 80.7)
- added J10: Encoder, Header:Conn_2x4, F.Cu at (117.1, 25.4)
- added J11: Conn_01x02_Male, Header:Conn_1x2, F.Cu at (-121.9, 56.5)
- added J12: Conn_01x02_Male, Header:Conn_1x2, F.Cu at (-119.4, 92.5)
- added J13: Conn_01x02_Male, Header:Conn_1x2, F.Cu at (-117.2, 126.9)
- added J14: Conn_01x02_Male, Header:Conn_1x2, F.Cu at (-73.7, 18.3)
- added J15: Conn_01x02_Male, Header:Conn_1x2, F.Cu at (-81.0, 57.9)
- added J16: Conn_01x02_Male, Header:Conn_1x2, F.Cu at (-78.1, 93.6)
- added J17: Conn_01x02_Male, Header:Conn_1x2, F.Cu at (-28.3, 19.2)
- added J18: Conn_01x02_Male, Header:Conn_1x2, F.Cu at (-38.7, 56.3)
- added J19: Conn_01x02_Male, Header:Conn_1x2, F.Cu at (-26.7, 89.4)
- added J2: TX_PORT, RS485:MTJ-642BX2, F.Cu at (33.6, 64.0)
- added J3: 87583-2010BLF, USB 2.0 Type A:87583-2010BLF, F.Cu at (199.1, 105.4)
- added J4: Conn_01x02_Male, Header:Conn_1x2, F.Cu at (-119.2, 21.7)
- added J5: GPIO Bank 0, Header:Conn_2x7, F.Cu at (98.6, 129.0)
- added J6: SPI 0, Header:Conn_2x4, F.Cu at (117.6, 129.0)
- added J7: Solenoid Power Selector, Header:Conn_1x3, F.Cu at (66.0, 30.7)
- added J8: GPIO Bank 1, Header:Conn_2x9, F.Cu at (149.9, 26.4)
- added J9: I2C 1-2, Header:Conn_2x5, F.Cu at (101.6, 24.9)
- added L1: 33u, 33 uH Inductor:LB3218T330K, F.Cu at (88.6, 74.7)
- added MOSFET1: SSM3K7002KFU, Toshiba MOSFET:SSM3K7002KFU, F.Cu at (-112.6, 13.1)
- added MOSFET10: SSM3K7002KFU, Toshiba MOSFET:SSM3K7002KFU, F.Cu at (-19.3, 80.3)
- added MOSFET2: SSM3K7002KFU, Toshiba MOSFET:SSM3K7002KFU, F.Cu at (-123.9, 49.8)
- added MOSFET3: SSM3K7002KFU, Toshiba MOSFET:SSM3K7002KFU, F.Cu at (-123.2, 82.3)
- added MOSFET4: SSM3K7002KFU, Toshiba MOSFET:SSM3K7002KFU, F.Cu at (-124.6, 111.8)
- added MOSFET5: SSM3K7002KFU, Toshiba MOSFET:SSM3K7002KFU, F.Cu at (-78.7, 21.3)
- added MOSFET6: SSM3K7002KFU, Toshiba MOSFET:SSM3K7002KFU, F.Cu at (-84.2, 48.3)
- added MOSFET7: SSM3K7002KFU, Toshiba MOSFET:SSM3K7002KFU, F.Cu at (-77.5, 82.6)
- added MOSFET8: SSM3K7002KFU, Toshiba MOSFET:SSM3K7002KFU, F.Cu at (-36.2, 21.2)
- added MOSFET9: SSM3K7002KFU, Toshiba MOSFET:SSM3K7002KFU, F.Cu at (-31.9, 46.6)
- added P1: J1B1211CCD, Ethernet:J1B1211CCD, F.Cu at (39.1, 89.9)
- added R1: 10, 10 Res:RNCP0603FTD10R0, F.Cu at (50.4, 73.7)
- added R2: 10, 10 Res:RNCP0603FTD10R0, F.Cu at (50.4, 70.6)
- added R3: 10, 10 Res:RNCP0603FTD10R0, F.Cu at (50.4, 56.4)
- added R4: 10, 10 Res:RNCP0603FTD10R0, F.Cu at (50.4, 53.3)
- added R5: 20k, 20K Res:SR1-0805-320, F.Cu at (96.7, 84.8)
- added R6: 10K, 10K Res:SR1-0603-310, F.Cu at (110.9, 76.2)
- added R7: 10K, 10K Res:SR1-0603-310, F.Cu at (98.6, 71.6)
- added U1: Teensy4.1, Teensy:Teensy41, F.Cu at (116.8, 56.9)
- added U2: 12V->5V, 12V5V Regulator:MC78M05CDTRKG, F.Cu at (43.4, 32.2)
- added U3: 12V->5V, 12V5V Regulator:MC78M05CDTRKG, F.Cu at (53.6, 32.2)
- added U4: 12V->5V, 12V5V Regulator:MC78M05CDTRKG, F.Cu at (33.3, 32.2)
- added U5: ISL83490IBZ, RS485 To UART:ISL83490IBZ, F.Cu at (55.5, 63.5)
- added U6: 74AXP2T3407GSX, Nexperia Level Shifter:74AXP2T3407GSX, F.Cu at (94.5, 45.7)
- added U7: 74AXP2T3407GSX, Nexperia Level Shifter:74AXP2T3407GSX, F.Cu at (97.5, 45.7)
- added U8: 12V->3.3V, 33SW:MIC2178-33YWM, F.Cu at (72.6, 73.7)
Routing:
- net +5V: track 0.00 -> 89.5 mm
- net /RS485_B_12V: track 0.00 -> 66.6 mm
- net /RS485_A_12V: track 0.00 -> 63.1 mm
- net GND: track 0.00 -> 28.5 mm, vias 0 -> 7
- net Net-(C6-Pad2): track 0.00 -> 17.5 mm
- net Net-(D2-Pad2): track 0.00 -> 17.2 mm
- net Net-(C4-Pad2): track 0.00 -> 15.4 mm
- net Net-(C5-Pad2): track 0.00 -> 15.0 mm
- net Net-(U5-Y): track 0.00 -> 8.96 mm
- net Net-(U5-A): track 0.00 -> 8.96 mm
- net Net-(U5-B): track 0.00 -> 7.45 mm
- net Net-(U5-Z): track 0.00 -> 7.34 mm
- net /Solenoid_Power: track 0.00 -> 4.57 mm
- added copper zone on F.Cu, net GND
Other:
- board outline added: 123.4 x 76.7 mm
- copper layers 0 -> 2
- board text added: "12V"
- board text added: "5V"
- board text added: "Literally Can't Mess This Up"

Commit message: Senior Update
Parts:
- added G***: LOGO, look of disapproval:Deep Fried Joe 2.5in, F.Cu at (365.8, -38.1)
- added G***: LOGO, look of disapproval:Cauchy Bowser Seal 1.5in, F.Cu at (246.4, 40.6)
- added G***: LOGO, look of disapproval:Deep Fried Joe 2in, F.Cu at (325.1, -43.2)
- added G***: LOGO, look of disapproval:test 1.5in, F.Cu at (411.5, 30.5)
- added G***: LOGO, look of disapproval:test 2in, F.Cu at (327.7, 40.6)
- added G***: LOGO, look of disapproval:Cauchy Bowser Seal 1in, F.Cu at (213.4, 33.0)
- moved C27 1.12 mm to (106.7, 73.7)
